File: PCB/hackpad.kicad_pcb (KiCad board)
At the start: 2 copper layers, 86.2 x 86.2 mm, 54 parts, among them SW1 Keyswitch, SW10 Keyswitch, SW11 Keyswitch, SW12 Keyswitch, SW13 EC05E1220203, SW14 EC05E1220203, SW2 Keyswitch, SW3 Keyswitch, SW4 Keyswitch, SW5 Keyswitch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

Commit message: case done
Parts:
- added G***: LOGO, assets:L1Simple, F.Cu at (70.0, 42.1)
- U2: footprint OLED_096_636:MODULE_DM-OLED096-636 -> OLED_096_636:AZ_OLED-096-SD1306
- moved U2 0.50 mm to (70.0, 42.3)
Routing:
- net COL0: track 103.6 -> 100.2 mm
- net GND: track 527.7 -> 526.9 mm
- net VCC: track 373.5 -> 372.8 mm
- net ROW3: track 104.2 -> 104.8 mm
- net SCL: track 17.1 -> 17.7 mm
- net SDA: track 17.7 -> 18.3 mm
